File: board/Board.kicad_pcb (KiCad board)
At the start: 2 copper layers, 54.9 x 61.9 mm, 57 parts, among them J10 CONN_01X03, J11 CONN_01X03, J12 CONN_01X02, J13 CONN_02X09, J14 CONN_02X04, SW1 SW_Push, SW2 SW_SPDT, SW3 SW_SPDT, U1 STM32F410RBTx, U2 LF33ABDT-TR, U3 ICM-20689, Y1 25 MHz, Y2 32.768 KHz

Commit message: ?
Parts:
- removed ? (x8), J10, J11: CONN_01X03, Pin_Headers:Pin_Header_Straight_1x03_Pitch2.54mm
- removed C1, C2: 20pF, Capacitors_SMD:C_0805_HandSoldering
- removed C10, C11, C12, C18, C24, C5, C7, C8: 100nF, Capacitors_SMD:C_0805_HandSoldering
- removed C16, C9: 4.7uF, Capacitors_SMD:C_0805_HandSoldering
- removed C17: 1uF, Capacitors_SMD:C_0805_HandSoldering
- removed C19: 0.1uF, Capacitors_SMD:C_0805_HandSoldering
- removed C20: 2.2uF, Capacitors_ThroughHole:CP_Radial_D5.0mm_P2.00mm
- removed C21: 10nF, Capacitors_SMD:C_0805_HandSoldering
- removed C22: 0.47uF, Capacitors_SMD:C_0805_HandSoldering
- removed C23: 2.2uF, Capacitors_SMD:C_0805_HandSoldering
- removed C3, C4: 1.5pF, Capacitors_SMD:C_0805_HandSoldering
- removed D1, D2: LED, LEDs:LED_0805
- removed G***: LOGO, Local_Prints:fedora-logo
- removed J12: CONN_01X02, Pin_Headers:Pin_Header_Straight_1x02_Pitch2.54mm
- removed J13: CONN_02X09, Pin_Headers:Pin_Header_Straight_2x09_Pitch2.54mm
- removed J14: CONN_02X04, Pin_Headers:Pin_Header_Straight_2x04_Pitch2.54mm
- removed JTAG: CONN_02X10, Pin_Headers:Pin_Header_Straight_2x10_Pitch2.54mm
- removed R1: 22, Resistors_SMD:R_0805_HandSoldering
- removed R10, R11, R2, R6, R7, R8, R9: 10K, Resistors_SMD:R_0805_HandSoldering
- removed R12: 220, Resistors_SMD:R_0805_HandSoldering
- removed R3, R4, R5: 0, Resistors_SMD:R_0805_HandSoldering
- removed SW1: SW_Push, Buttons_Switches_ThroughHole:SW_PUSH_6mm
- removed SW2, SW3: SW_SPDT, Pin_Headers:Pin_Header_Straight_1x03_Pitch2.54mm
- removed U1: STM32F410RBTx, Housings_QFP:LQFP-64_10x10mm_Pitch0.5mm
- removed U2: LF33ABDT-TR, TO_SOT_Packages_SMD:TO-252-2Lead
- removed U3: ICM-20689, Housings_DFN_QFN:QFN-24-1EP_4x4mm_Pitch0.5mm
- removed Y1: 25 MHz, Crystals:Crystal_HC49-U_Vertical
- removed Y2: 32.768 KHz, Crystals:Crystal_SMD_5032-2pin_5.0x3.2mm_HandSoldering
Routing:
- net VCC: track 225.9 -> 0.00 mm, vias 6 -> 0
- net PC8: track 113.8 -> 0.00 mm, vias 12 -> 0
- net NRST: track 87.9 -> 0.00 mm, vias 6 -> 0
- net PC9: track 78.9 -> 0.00 mm, vias 2 -> 0
- net GND: track 76.8 -> 0.00 mm, vias 21 -> 0
- net PB11: track 69.3 -> 0.00 mm, vias 2 -> 0
- net PC11: track 67.2 -> 0.00 mm, vias 6 -> 0
- net PC12: track 66.7 -> 0.00 mm, vias 10 -> 0
- net PB5: track 62.7 -> 0.00 mm, vias 2 -> 0
- net Net-(D1-Pad2): track 48.8 -> 0.00 mm, vias 6 -> 0
- net PWM_OUTPUT_1: track 46.7 -> 0.00 mm
- net PWM_OUTPUT_2: track 44.8 -> 0.00 mm
- net PC13: track 44.2 -> 0.00 mm, vias 2 -> 0
- net UART_TX: track 43.9 -> 0.00 mm, vias 6 -> 0
- net UART_RX: track 43.6 -> 0.00 mm, vias 6 -> 0
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- removed copper zone on B.Cu, net GND
Other:
- board outline removed
- rule pad_to_mask_clearance: 0.2 -> 0
- board text removed: "0"
- board text removed: "1"
- board text removed: "2"
- board text removed: "3"
- board text removed: "4"
- board text removed: "BOOT"
- board text removed: "GPIO"
- board text removed: "I2C"
- board text removed: "Input"
- board text removed: "M'Copter Rev 1.0"
- board text removed: "Output"
- board text removed: "PWR"
- board text removed: "RF24"
- board text removed: "Reset"
- board text removed: "UART"

Commit message: pcb rev2, work in progress
Parts:
- added C1: 20pF, Capacitors_SMD:C_0805_HandSoldering, F.Cu at (113.9, 90.2)
- added C10: 100nF, Capacitors_SMD:C_0805_HandSoldering, F.Cu at (118.2, 90.2)
- added C11: 100nF, Capacitors_SMD:C_0805_HandSoldering, F.Cu at (124.3, 96.5)
- added C12: 100nF, Capacitors_SMD:C_0805_HandSoldering, F.Cu at (123.7, 80.0)
- added C16: 4.7uF, Capacitors_SMD:C_0805_HandSoldering, F.Cu at (123.7, 77.5)
- added C17: 1uF, Capacitors_SMD:C_0805_HandSoldering, F.Cu at (138.8, 84.0)
- added C18: 100nF, Capacitors_SMD:C_0805_HandSoldering, F.Cu at (144.3, 84.0)
- added C19: 0.1uF, Capacitors_SMD:C_0805_HandSoldering, F.Cu at (122.7, 64.1)
- added C2: 20pF, Capacitors_SMD:C_0805_HandSoldering, F.Cu at (116.0, 90.2)
- added C20: 2.2uF, Capacitors_ThroughHole:CP_Radial_D5.0mm_P2.00mm, F.Cu at (122.4, 68.1)
- added C21: 10nF, Capacitors_SMD:C_0805_HandSoldering, F.Cu at (117.0, 108.7)
- added C22: 0.47uF, Capacitors_SMD:C_0805_HandSoldering, F.Cu at (124.1, 109.7)
- added C23: 2.2uF, Capacitors_SMD:C_0805_HandSoldering, F.Cu at (116.3, 113.2)
- added C24: 100nF, Capacitors_SMD:C_0805_HandSoldering, F.Cu at (124.0, 113.5)
- added C5: 100nF, Capacitors_SMD:C_0805_HandSoldering, F.Cu at (215.2, 138.7)
- added C7: 100nF, Capacitors_SMD:C_0805_HandSoldering, F.Cu at (117.3, 82.9)
- added C8: 100nF, Capacitors_SMD:C_0805_HandSoldering, F.Cu at (132.8, 96.1)
- added C9: 4.7uF, Capacitors_SMD:C_0805_HandSoldering, F.Cu at (185.4, 117.3)
- added D1: LED, LEDs:LED_0805, F.Cu at (208.9, 155.3)
- added D2: LED, LEDs:LED_0805, F.Cu at (109.4, 72.1)
- added J1: CONN_02X10, Connect:IDC_Header_Straight_20pins, F.Cu at (149.4, 68.4)
- added J10: CONN_01X03, Pin_Headers:Pin_Header_Straight_1x03_Pitch2.54mm, F.Cu at (181.1, 150.1)
- added J11: CONN_01X03, Pin_Headers:Pin_Header_Straight_1x03_Pitch2.54mm, F.Cu at (215.3, 121.9)
- added J12: CONN_01X02, Pin_Headers:Pin_Header_Straight_1x02_Pitch2.54mm, F.Cu at (191.2, 150.1)
- added J13: CONN_02X09, Pin_Headers:Pin_Header_Straight_2x09_Pitch2.54mm, F.Cu at (156.2, 125.0)
- added J15: GS3, Connect:GS3, F.Cu at (203.9, 153.7)
- added J16: GS3, Connect:GS3, F.Cu at (208.8, 145.0)
- added J17: GS3, Connect:GS3, F.Cu at (240.4, 114.7)
- added J18: GS2, Connect:GS2, F.Cu at (175.3, 144.3)
- added J19: CONN_01X01, Pin_Headers:Pin_Header_Straight_1x01_Pitch2.54mm, F.Cu at (207.6, 133.7)
- added J2: CONN_01X03, Pin_Headers:Pin_Header_Straight_1x03_Pitch2.54mm, F.Cu at (167.4, 80.9)
- added J3: CONN_01X03, Pin_Headers:Pin_Header_Straight_1x03_Pitch2.54mm, F.Cu at (171.8, 80.9)
- added J4: CONN_01X03, Pin_Headers:Pin_Header_Straight_1x03_Pitch2.54mm, F.Cu at (176.3, 81.2)
- added J5: CONN_01X03, Pin_Headers:Pin_Header_Straight_1x03_Pitch2.54mm, F.Cu at (180.9, 81.3)
- added J6: CONN_01X03, Pin_Headers:Pin_Header_Straight_1x03_Pitch2.54mm, F.Cu at (167.4, 90.8)
- added J7: CONN_01X03, Pin_Headers:Pin_Header_Straight_1x03_Pitch2.54mm, F.Cu at (171.9, 90.6)
- added J8: CONN_01X03, Pin_Headers:Pin_Header_Straight_1x03_Pitch2.54mm, F.Cu at (176.3, 91.6)
- added J9: CONN_01X03, Pin_Headers:Pin_Header_Straight_1x03_Pitch2.54mm, F.Cu at (180.9, 91.9)
- added R1: 22, Resistors_SMD:R_0805_HandSoldering, F.Cu at (220.2, 138.6)
- added R10: 10K, Resistors_SMD:R_0805_HandSoldering, F.Cu at (203.8, 158.8)
- added R11: 10K, Resistors_SMD:R_0805_HandSoldering, F.Cu at (236.9, 119.8)
- added R12: 220, Resistors_SMD:R_0805_HandSoldering, F.Cu at (114.0, 72.2)
- added R2: 10K, Resistors_SMD:R_0805_HandSoldering, F.Cu at (230.3, 129.8)
- added R3: 0, Resistors_SMD:R_0805_HandSoldering, F.Cu at (220.3, 144.1)
- added R4: 62K, Resistors_SMD:R_0805_HandSoldering, F.Cu at (215.1, 144.2)
- added R5: 22K, Resistors_SMD:R_0805_HandSoldering, F.Cu at (225.1, 131.7)
- added R6: 10K, Resistors_SMD:R_0805_HandSoldering, F.Cu at (225.4, 137.2)
- added R7: 10K, Resistors_SMD:R_0805_HandSoldering, F.Cu at (214.5, 149.7)
- added R8: 10K, Resistors_SMD:R_0805_HandSoldering, F.Cu at (209.3, 150.1)
- added R9: 10K, Resistors_SMD:R_0805_HandSoldering, F.Cu at (236.9, 125.3)
- added SW1: SW_Push, Buttons_Switches_ThroughHole:SW_PUSH_6mm, F.Cu at (207.9, 105.3)
- added U1: STM32F410RBTx, Housings_QFP:LQFP-64_10x10mm_Pitch0.5mm, F.Cu at (128.0, 88.0)
- added U2: LF33ABDT-TR, TO_SOT_Packages_SMD:TO-252-2Lead, F.Cu at (112.6, 66.9)
- added U3: ICM-20689, Housings_DFN_QFN:QFN-24-1EP_4x4mm_Pitch0.5mm, F.Cu at (124.3, 103.9)
- added U4: SN74LVC1G04, TO_SOT_Packages_SMD:SOT-23-5_HandSoldering, F.Cu at (225.8, 110.7)
- added Y1: 25 MHz, Crystals:Crystal_HC49-U_Vertical, F.Cu at (109.5, 88.9)
