File: board/Board.kicad_pcb (KiCad board)
At the start: 2 copper layers, 58.5 x 58.5 mm, 63 parts, among them J1 GS3, J10 CONN_01X03, J11 CONN_01X03, J12 GS3, J13 GS3, J14 CONN_01X02, J15 CONN_01X03, J16 GS2, J17 CONN_01X01, J2 CONN_02X04, J3 CONN_01X03, J4 CONN_01X03, J5 CONN_01X03, J6 CONN_01X03, J7 CONN_01X03, J8 CONN_01X03, J9 CONN_01X03, SW1 SW_Push, U1 STM32F410RBTx, U2 SN74LVC1G04, U3 LF33ABDT-TR, U4 ICM-20689, U5 MAG3110, U6 MS5637, Y1 25 MHz

Commit message: more routes
Routing:
- net VCC: track 104.2 -> 143.9 mm
- net JTCK: track 0.00 -> 24.7 mm
- net JTMS: track 0.00 -> 21.0 mm, vias 0 -> 2
- net JTDO: track 0.00 -> 17.4 mm
- net JTRST: track 0.00 -> 14.0 mm
- net JTDI: track 0.00 -> 13.8 mm
Changed lines of the file:
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@@
   (general
     (links 151)
-    (no_connects 103)
-    (area 95.681217 65.689424 154.310576 124.300001)
+    (no_connects 98)
+    (area 90.442857 64.575 159.557143 125.275)
     (thickness 1.6)
     (drawings 8)
-    (tracks 122)
+    (tracks 162)
     (zones 0)
     (modules 63)
@@
   (gr_arc (start 150 70) (end 150.2 65.75) (angle 90) (layer Edge.Cuts) (width 0.1))
   (gr_arc (start 100 70) (end 95.75 69.7) (angle 90) (layer Edge.Cuts) (width 0.1))
-  (segment (start 138.5 91.6) (end 137.95 91.6) (width 0.25) (layer F.Cu) (net 1) (status C00000))
-  (segment (start 137.95 91.6) (end 136.75 90.4) (width 0.25) (layer F.Cu) (net 1) (status 400000))
-  (segment (start 136.75 90.4) (end 134.75 90.4) (width 0.25) (layer F.Cu) (net 1) (status 800000))
-  (segment (start 134.45 102.5) (end 133.45 102.5) (width 0.25) (layer F.Cu) (net 1) (status 400000))
-  (segment (start 132.05 101.1) (end 132.05 99.6) (width 0.25) (layer F.Cu) (net 1) (status 800000))
+  (segment (start 138.5 91.6) (end 137.95 91.6) (width 0.25) (layer F.Cu) (net 1))
+  (segment (start 137.95 91.6) (end 136.75 90.4) (width 0.25) (layer F.Cu) (net 1))
+  (segment (start 136.75 90.4) (end 134.75 90.4) (width 0.25) (layer F.Cu) (net 1))
+  (segment (start 134.45 102.5) (end 133.45 102.5) (width 0.25) (layer F.Cu) (net 1))
+  (segment (start 132.05 101.1) (end 132.05 99.6) (width 0.25) (layer F.Cu) (net 1))
   (segment (start 133.45 102.5) (end 132.05 101.1) (width 0.25) (layer F.Cu) (net 1))
-  (segment (start 131.6 105.8) (end 132.95 105.8) (width 0.25) (layer F.Cu) (net 1) (status 400000))
+  (segment (start 131.6 105.8) (end 132.95 105.8) (width 0.25) (layer F.Cu) (net 1))
   (via (at 132.95 105.8) (size 0.6) (drill 0.4) (layers F.Cu B.Cu) (net 1))
   (segment (start 123.95 102.35) (end 123.95 102.1) (width 0.25) (layer F.Cu) (net 1))
@@
   (segment (start 119.35 93.4) (end 120.35 92.4) (width 0.25) (layer F.Cu) (net 3))
   (segment (start 112 93.4) (end 116.8 93.4) (width 0.25) (layer F.Cu) (net 3))
-  (segment (start 138.5 89.1) (end 136.95 89.1) (width 0.25) (layer F.Cu) (net 5) (status 400000))
-  (segment (start 136.15 89.9) (end 134.75 89.9) (width 0.25) (layer F.Cu) (net 5) (status 800000))
+  (segment (start 134.75 89.9) (end 131.075 89.9) (width 0.25) (layer F.Cu) (net 5))
+  (segment (start 131.075 89.9) (end 127.7875 93.1875) (width 0.25) (layer F.Cu) (net 5))
+  (segment (start 122.85 89.9) (end 124.5 89.9) (width 0.25) (layer F.Cu) (net 5))
+  (segment (start 124.5 89.9) (end 127.7875 93.1875) (width 0.25) (layer F.Cu) (net 5))
+  (segment (start 132.55 97.95) (end 132.55 99.6) (width 0.25) (layer F.Cu) (net 5))
+  (segment (start 127.7875 93.1875) (end 132.55 97.95) (width 0.25) (layer F.Cu) (net 5))
+  (segment (start 128 77.7) (end 122.85 77.7) (width 0.25) (layer F.Cu) (net 5))
+  (segment (start 129.7 76) (end 128 77.7) (width 0.25) (layer F.Cu) (net 5))
+  (segment (start 132.1 76) (end 129.7 76) (width 0.25) (layer F.Cu) (net 5))
+  (segment (start 122.85 77.7) (end 124.35 76.2) (width 0.25) (layer F.Cu) (net 5))
+  (segment (start 121.5 80.25) (end 121.5 79.05) (width 0.25) (layer F.Cu) (net 5))
+  (segment (start 124.35 76.2) (end 124.35 74.75) (width 0.25) (layer F.Cu) (net 5))
+  (segment (start 121.5 79.05) (end 122.85 77.7) (width 0.25) (layer F.Cu) (net 5))
+  (segment (start 138.5 89.1) (end 136.95 89.1) (width 0.25) (layer F.Cu) (net 5))
+  (segment (start 136.15 89.9) (end 134.75 89.9) (width 0.25) (layer F.Cu) (net 5))
   (segment (start 136.95 89.1) (end 136.15 89.9) (width 0.25) (layer F.Cu) (net 5))
-  (segment (start 132.55 99.6) (end 132.55 100.65) (width 0.25) (layer F.Cu) (net 5) (status 400000))
-  (segment (start 135.85 101.4) (end 136.95 102.5) (width 0.25) (layer F.Cu) (net 5) (status 800000))
+  (segment (start 132.55 99.6) (end 132.55 100.65) (width 0.25) (layer F.Cu) (net 5))
+  (segment (start 132.55 100.65) (end 133.3 101.4) (width 0.25) (layer F.Cu) (net 5))
   (segment (start 133.3 101.4) (end 135.85 101.4) (width 0.25) (layer F.Cu) (net 5))
-  (segment (start 132.55 100.65) (end 133.3 101.4) (width 0.25) (layer F.Cu) (net 5))
+  (segment (start 135.85 101.4) (end 136.95 102.5) (width 0.25) (layer F.Cu) (net 5))
   (segment (start 118.95 101) (end 119.2 101) (width 0.25) (layer F.Cu) (net 5))
   (segment (start 119.2 101) (end 121.95 103.75) (width 0.25) (layer F.Cu) (net 5))
@@
   (segment (start 121.65 80.25) (end 124.1 82.7) (width 0.25) (layer F.Cu) (net 5))
   (segment (start 113.25 80.25) (end 118.65 80.25) (width 0.25) (layer F.Cu) (net 5))
-  (segment (start 118.65 80.25) (end 121.65 80.25) (width 0.25) (layer F.Cu) (net 5))
+  (segment (start 118.65 80.25) (end 121.5 80.25) (width 0.25) (layer F.Cu) (net 5))
+  (segment (start 121.5 80.25) (end 121.65 80.25) (width 0.25) (layer F.Cu) (net 5))
   (segment (start 124.1 82.7) (end 124.1 85.6) (width 0.25) (layer F.Cu) (net 5))
   (segment (start 124.1 85.6) (end 125.05 86.55) (width 0.25) (layer F.Cu) (net 5))
@@
   (segment (start 104.1 81.35) (end 104.1 83.5) (width 0.25) (layer F.Cu) (net 13))
   (segment (start 104.1 83.5) (end 104.25 83.65) (width 0.25) (layer F.Cu) (net 13))
+  (segment (start 132.55 87.7) (end 132.55 82.75) (width 0.25) (layer F.Cu) (net 15))
+  (segment (start 133.535 72.025) (end 132.1 73.46) (width 0.25) (layer F.Cu) (net 15))
+  (segment (start 137.9 72.025) (end 133.535 72.025) (width 0.25) (layer F.Cu) (net 15))
+  (segment (start 138.45 72.575) (end 137.9 72.025) (width 0.25) (layer F.Cu) (net 15))
+  (segment (start 138.45 76.85) (end 138.45 72.575) (width 0.25) (layer F.Cu) (net 15))
+  (segment (start 132.55 82.75) (end 138.45 76.85) (width 0.25) (layer F.Cu) (net 15))
+  (segment (start 134.64 76) (end 134.64 77.46) (width 0.25) (layer F.Cu) (net 16))
+  (segment (start 129.05 83.05) (end 129.05 87.7) (width 0.25) (layer F.Cu) (net 16))
+  (segment (start 134.64 77.46) (end 129.05 83.05) (width 0.25) (layer F.Cu) (net 16))
+  (segment (start 129.55 87.7) (end 129.55 83.375) (width 0.25) (layer F.Cu) (net 17))
+  (segment (start 135.9 74.72) (end 134.64 73.46) (width 0.25) (layer F.Cu) (net 17))
+  (segment (start 135.9 77.025) (end 135.9 74.72) (width 0.25) (layer F.Cu) (net 17))
+  (segment (start 129.55 83.375) (end 135.9 77.025) (width 0.25) (layer F.Cu) (net 17))
+  (segment (start 137.18 76) (end 137.18 77.245) (width 0.25) (layer F.Cu) (net 18))
+  (segment (start 132.05 82.375) (end 132.05 87.7) (width 0.25) (layer F.Cu) (net 18))
+  (segment (start 137.18 77.245) (end 132.05 82.375) (width 0.25) (layer F.Cu) (net 18))
+  (segment (start 139.72 76) (end 139.72 76.63) (width 0.25) (layer F.Cu) (net 19))
+  (segment (start 139.72 76.63) (end 133.075 83.275) (width 0.25) (layer F.Cu) (net 19))
+  (segment (start 132.275 90.9) (end 134.75 90.9) (width 0.25) (layer F.Cu) (net 19))
+  (segment (start 132.075 90.7) (end 132.275 90.9) (width 0.25) (layer F.Cu) (net 19))
+  (via (at 132.075 90.7) (size 0.6) (drill 0.4) (layers F.Cu B.Cu) (net 19))
+  (segment (start 132.075 90.25) (end 132.075 90.7) (width 0.25) (layer B.Cu) (net 19))
+  (segment (start 133.075 89.25) (end 132.075 90.25) (width 0.25) (layer B.Cu) (net 19))
+  (via (at 133.075 89.25) (size 0.6) (drill 0.4) (layers F.Cu B.Cu) (net 19))
+  (segment (start 133.075 83.275) (end 133.075 89.25) (width 0.25) (layer F.Cu) (net 19))
+  (segment (start 139.72 76) (end 139.72 76.405) (width 0.25) (layer F.Cu) (net 19))
   (segment (start 100.2 86.3) (end 99.6 86.3) (width 0.25) (layer F.Cu) (net 41))
   (segment (start 99.6 86.3) (end 99.4 86.5) (width 0.25) (layer F.Cu) (net 41))
@@
   (segment (start 119.6 90.95) (end 120.55 91.9) (width 0.25) (layer F.Cu) (net 42))
   (segment (start 120.55 91.9) (end 122.85 91.9) (width 0.25) (layer F.Cu) (net 42))
-  (segment (start 102.05 92.3) (end 104.7 92.3) (width 0.25) (layer F.Cu) (net 45) (status 400000))
-  (segment (start 121.55 93.4) (end 122.85 93.4) (width 0.25) (layer F.Cu) (net 45) (status 800000))
+  (segment (start 102.05 92.3) (end 104.7 92.3) (width 0.25) (layer F.Cu) (net 45))
+  (segment (start 121.55 93.4) (end 122.85 93.4) (width 0.25) (layer F.Cu) (net 45))
   (segment (start 118.6 96.35) (end 121.55 93.4) (width 0.25) (layer F.Cu) (net 45))
   (via (at 118.6 96.35) (size 0.6) (drill 0.4) (layers F.Cu B.Cu) (net 45))
@@
     (polygon
       (pts
-        (xy 153.2 125.25) (xy 97.8 125.25) (xy 97.8 69.85) (xy 153.2 69.85)
+        (xy 152.7 122.7) (xy 97.3 122.7) (xy 97.3 67.3) (xy 152.7 67.3)
       )
     )

Commit message: wip
Parts:
- moved C15 9.05 mm to (107.9, 117.7)
- moved C17 9.05 mm to (107.8, 120.2)
- moved U5 9.05 mm to (112.8, 119.8)
- moved C20 6.94 mm to (120.2, 117.1)
- moved U4 6.72 mm to (119.2, 111.2)
- moved C22 6.49 mm to (123.5, 111.2)
- moved C18 6.39 mm to (117.5, 117.0)
- moved C24 4.80 mm to (125.5, 111.2)
- moved J15 3.57 mm to (146.9, 109.3)
- moved J11 3.41 mm to (143.0, 109.3)
- moved C9 1.90 mm to (123.3, 102.3)
Routing:
- net I2C2_SDA: track 0.00 -> 37.6 mm, vias 0 -> 6
- net ICM_SPI_MISO: track 0.00 -> 28.0 mm, vias 0 -> 4
- net I2C2_SCL: track 0.00 -> 20.4 mm
- net ICM_INT: track 0.00 -> 19.3 mm, vias 0 -> 2
- net ICM_SPI_SCK: track 0.00 -> 15.9 mm, vias 0 -> 2
- net VCC: track 143.9 -> 158.8 mm
- net ICM_SPI_CS: track 0.00 -> 14.4 mm
- net GND: track 45.5 -> 57.3 mm, vias 9 -> 13
- net Net-(C20-Pad1): track 0.00 -> 3.01 mm

Commit message: backup
Parts:
- moved C19 23.1 mm to (112.8, 111.1), turned to 0 degrees
- moved C21 20.5 mm to (112.8, 113.1), turned to 0 degrees
- moved C23 17.8 mm to (112.8, 115.1), turned to 0 degrees
- moved C15 1.13 mm to (107.7, 118.8)
- moved C17 0.90 mm to (107.8, 121.1)
Routing:
- net VCC: track 158.8 -> 163.9 mm
- net GND: track 57.3 -> 61.4 mm

Commit message: outing mag
Parts:
- moved C15 1.84 mm to (106.5, 117.4)
- moved C17 1.29 mm to (106.5, 120.7)
- moved U5 0.89 mm to (112.3, 119.1), turned to 270 degrees
Routing:
- net MAG_INT: track 0.00 -> 34.3 mm, vias 0 -> 4
- net VCC: track 163.9 -> 189.5 mm, vias 0 -> 2
- net I2C2_SCL: track 20.4 -> 45.9 mm, vias 0 -> 2
- net ICM_SPI_MOSI: track 0.00 -> 18.3 mm, vias 0 -> 2
- net I2C2_SDA: track 37.6 -> 55.2 mm
- net GND: track 61.4 -> 77.1 mm, vias 13 -> 20
- net Net-(C15-Pad1): track 0.00 -> 4.64 mm
- net Net-(C17-Pad1): track 0.00 -> 4.26 mm

Commit message: finished routing
Parts:
- moved R1 32.3 mm to (109.3, 109.2), turned to 270 degrees
- moved D1 30.9 mm to (110.4, 105.8), turned to 0 degrees
- moved SW1 8.25 mm to (106.7, 112.4), turned to 180 degrees
- moved J11 7.25 mm to (149.5, 106.1), turned to 270 degrees
- moved J6 6.15 mm to (145.8, 97.5)
- moved J5 5.10 mm to (145.8, 95.0)
- moved J15 4.06 mm to (149.5, 112.5), turned to 270 degrees
- moved J4 4.00 mm to (145.8, 92.5)
- moved J3 2.90 mm to (145.8, 90.0)
- moved U2 2.78 mm to (135.8, 119.2)
- moved J7 2.00 mm to (145.7, 78.3)
- moved J13 1.97 mm to (142.6, 117.6), turned to 90 degrees
- moved R3 1.54 mm to (106.6, 101.0)
- moved J1 1.50 mm to (106.6, 103.3)
- moved J10 1.30 mm to (145.7, 85.8)
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Routing:
- net I2C1_SCL: track 0.00 -> 61.0 mm, vias 0 -> 7
- net I2C1_SDA: track 0.00 -> 58.5 mm, vias 0 -> 6
- net UART_TX: track 0.00 -> 50.7 mm, vias 0 -> 6
- net Net-(R3-Pad2): track 0.00 -> 45.1 mm, vias 0 -> 4
- net UART_RX: track 0.00 -> 44.8 mm, vias 0 -> 4
- net Net-(C3-Pad1): track 0.00 -> 40.9 mm, vias 0 -> 2
- net Net-(R6-Pad1): track 0.00 -> 32.6 mm, vias 0 -> 6
- net VCC: track 189.5 -> 216.6 mm
- net PWM_INPUT_2: track 0.00 -> 26.8 mm
- net PWM_OUTPUT_1: track 0.00 -> 26.6 mm, vias 0 -> 2
- net PWM_OUTPUT_2: track 0.00 -> 24.7 mm, vias 0 -> 2
- net PWM_OUTPUT_3: track 0.00 -> 23.9 mm, vias 0 -> 2
- net PWM_INPUT_1: track 0.00 -> 23.8 mm, vias 0 -> 2
- net Net-(D1-Pad2): track 0.00 -> 22.4 mm, vias 0 -> 4
- net PWM_OUTPUT_4: track 0.00 -> 22.3 mm, vias 0 -> 2
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